File: hardware/SEBC_Hardware/SEBC_Hardware.sch (KiCad schematic (older format))
At the start: 1 part

Commit message: :electric_plug:  Add sensor
Parts:
- added J?: AudioJack2_Ground, symbol Connector:AudioJack2_Ground
- added R? (x2): 10 k, symbol Device:R
Connections:
- wire segments 0 -> 4
Changed lines of the file:
@@
 	1    0    0    -1
 $EndComp
+$Comp
+L Connector:AudioJack2_Ground J?
+U 1 1 5B568116
+P 6200 1700
+F 0 "J?" H 5967 1679 50  0000 R CNN
+F 1 "AudioJack2_Ground" H 5967 1770 50  0000 R CNN
+F 2 "" H 6200 1700 50  0001 C CNN
+F 3 "~" H 6200 1700 50  0001 C CNN
+	1    6200 1700
+	-1   0    0    1
+$EndComp
+$Comp
+L Device:R R?
+U 1 1 5B568250
+P 5200 1400
+F 0 "R?" V 4993 1400 50  0000 C CNN
+F 1 "10 k" V 5084 1400 50  0000 C CNN
+F 2 "" V 5130 1400 50  0001 C CNN
+F 3 "~" H 5200 1400 50  0001 C CNN
+	1    5200 1400
+	0    1    1    0
+$EndComp
+$Comp
+L Device:R R?
+U 1 1 5B56831A
+P 5650 1400
+F 0 "R?" V 5443 1400 50  0000 C CNN
+F 1 "10 k" V 5534 1400 50  0000 C CNN
+F 2 "" V 5580 1400 50  0001 C CNN
+F 3 "~" H 5650 1400 50  0001 C CNN
+	1    5650 1400
+	0    1    1    0
+$EndComp
+Wire Wire Line
+	5350 1400 5400 1400
+Wire Wire Line
+	6000 1700 5400 1700
+Wire Wire Line
+	5400 1700 5400 1400
+Connection ~ 5400 1400
+Wire Wire Line
+	5400 1400 5500 1400
 $EndSCHEMATC

Commit message: :electric_plug: Add mews plugs
Parts:
- added C? (x2): 100 uF, symbol Device:CP
- added C?: C, symbol Device:C
- added C? (x2): 10uF, symbol Device:CP1
- added D?: DIODE, symbol pspice:DIODE
- added D? (x2): LED_ALT, symbol Device:LED_ALT
- added D?: D_Zener_ALT, symbol Device:D_Zener_ALT
- added J?: AudioJack2_Ground, symbol Connector:AudioJack2_Ground
- added J?: Barrel_Jack_Switch, symbol Connector:Barrel_Jack_Switch
- added J?: Micro_SD_Card, symbol Connector:Micro_SD_Card
- added R? (x3): 10 k, symbol Device:R
- added R? (x2): 1 k, symbol Device:R
- added R?: R, symbol Device:R
- added SW? (x2): SW_Push, symbol Switch:SW_Push
- added U?: L7805, symbol Regulator_Linear:L7805
Connections:
- net labels added: +3.3V, +5V, Boot, CLK, DAT0, GND, LED_01, LED_02, Reset, SD1, SD2, SENSOR_C_A, SENSOR_C_B
- wire segments 4 -> 85
- no-connect marks 0 -> 2

Commit message: :book: ESP8266 Kicad Library
Parts:
- added C? (x2): C, symbol Device:C
- added J? (x2): Conn_01x02, symbol Connector_Generic:Conn_01x02
- added R? (x4): R, symbol Device:R
- added U? (x2): 4N25, Package_DIP:DIP-6_W7.62mm, symbol Isolator:4N25
- added U?: 4051, symbol 4xxx:4051
Connections:
- net labels added: A0, A1, A2, INN_E, SENSOR_T_A, SENSOR_T_B, S_MUX
- wire segments 85 -> 137

Commit message: :construction:  Adicionando MicroSD
Parts:
- C?: value C -> 100 n
- C? (x2): value C -> 100 u
- R?: value R -> 1k
- R? (x2): value R -> 10k
- R? (x2): value R -> 220k
Changed lines of the file:
@@
 Wire Wire Line
 	6900 1300 6900 1350
-$Comp
-L power:+5V #PWR?
-U 1 1 5B580063
-P 5400 1200
-F 0 "#PWR?" H 5400 1050 50  0001 C CNN
-F 1 "+5V" H 5415 1373 50  0000 C CNN
-F 2 "" H 5400 1200 50  0001 C CNN
-F 3 "" H 5400 1200 50  0001 C CNN
-	1    5400 1200
-	1    0    0    -1
-$EndComp
 Wire Wire Line
 	5400 1200 5400 1300
@@
 P 5850 2400
 F 0 "R?" V 5643 2400 50  0000 C CNN
-F 1 "R" V 5734 2400 50  0000 C CNN
+F 1 "1k" V 5734 2400 50  0000 C CNN
 F 2 "" V 5780 2400 50  0001 C CNN
 F 3 "~" H 5850 2400 50  0001 C CNN
@@
 P 6600 2400
 F 0 "C?" V 6348 2400 50  0000 C CNN
-F 1 "C" V 6439 2400 50  0000 C CNN
+F 1 "100 n" V 6439 2400 50  0000 C CNN
 F 2 "" H 6638 2250 50  0001 C CNN
 F 3 "~" H 6600 2400 50  0001 C CNN
@@
 P 6600 5550
 F 0 "R?" H 6670 5596 50  0000 L CNN
-F 1 "R" H 6670 5505 50  0000 L CNN
+F 1 "10k" H 6670 5505 50  0000 L CNN
 F 2 "" V 6530 5550 50  0001 C CNN
 F 3 "~" H 6600 5550 50  0001 C CNN
@@
 P 7000 5550
 F 0 "C?" H 7115 5596 50  0000 L CNN
-F 1 "C" H 7115 5505 50  0000 L CNN
+F 1 "100 u" H 7115 5505 50  0000 L CNN
 F 2 "" H 7038 5400 50  0001 C CNN
 F 3 "~" H 7000 5550 50  0001 C CNN
@@
 P 5300 5100
 F 0 "R?" V 5093 5100 50  0000 C CNN
-F 1 "R" V 5184 5100 50  0000 C CNN
+F 1 "220k" V 5184 5100 50  0000 C CNN
 F 2 "" V 5230 5100 50  0001 C CNN
 F 3 "~" H 5300 5100 50  0001 C CNN
@@
 P 9800 5550
 F 0 "R?" H 9870 5596 50  0000 L CNN
-F 1 "R" H 9870 5505 50  0000 L CNN
+F 1 "10k" H 9870 5505 50  0000 L CNN
 F 2 "" V 9730 5550 50  0001 C CNN
 F 3 "~" H 9800 5550 50  0001 C CNN
@@
 P 10200 5550
 F 0 "C?" H 10315 5596 50  0000 L CNN
-F 1 "C" H 10315 5505 50  0000 L CNN
+F 1 "100 u" H 10315 5505 50  0000 L CNN
 F 2 "" H 10238 5400 50  0001 C CNN
 F 3 "~" H 10200 5550 50  0001 C CNN
@@
 P 8500 5100
 F 0 "R?" V 8293 5100 50  0000 C CNN
-F 1 "R" V 8384 5100 50  0000 C CNN
+F 1 "220k" V 8384 5100 50  0000 C CNN
 F 2 "" V 8430 5100 50  0001 C CNN
 F 3 "~" H 8500 5100 50  0001 C CNN
@@
 Text Label 2300 5100 2    50   ~ 0
 SENSOR_C_B
+Text Label 5400 1200 2    50   ~ 0
+Reset
 $EndSCHEMATC

Commit message: :construction_worker: PCB
Parts:
- removed C? (x2): 100 u, symbol Device:C
- removed J? (x2): AudioJack2_Ground, symbol Connector:AudioJack2_Ground
- removed J? (x2): Conn_01x02, symbol Connector_Generic:Conn_01x02
- added C5, C7: 10uF, Capacitor_THT:CP_Radial_D5.0mm_P2.50mm, symbol Device:CP1
- added J2, J3, J5, J6: Conn_01x01_Female, Connector:Banana_Jack_1Pin, symbol Connector:Conn_01x01_Female
- added J4, J7: AudioJack2_Ground_Switch, ESP8266:JACKAUDIO_P2, symbol Connector:AudioJack2_Ground_Switch
- C1, C2, C4: renamed from C?; footprint (none) -> Capacitor_THT:CP_Radial_D5.0mm_P2.50mm
- C3, C6: renamed from C?; footprint (none) -> Capacitor_THT:CP_Radial_D8.0mm_P3.50mm
- D1, D2: renamed from D?; footprint (none) -> Diode_THT:D_A-405_P7.62mm_Horizontal
- D3, D4: renamed from D?; footprint (none) -> LED_THT:LED_D5.0mm
- J1: renamed from J?; footprint (none) -> Connector_BarrelJack:BarrelJack_Horizontal
- J8: renamed from J?; footprint (none) -> ESP8266:microSD
- R1, R10, R11, R12, R2, R3, R4, R5, R6, R7, R8, R9: renamed from R?; footprint (none) -> Resistor_THT:R_Axial_DIN0207_L6.3mm_D2.5mm_P7.62mm_Horizontal
- SW1, SW2: renamed from SW?; footprint (none) -> ESP8266:push_button
- U1: renamed from U?; footprint (none) -> ESP8266:nodmcu
- U2: renamed from U?; footprint (none) -> Package_TO_SOT_THT:TO-220-3_Vertical
- U3: renamed from U?; footprint (none) -> Package_DIP:DIP-16_W7.62mm
- gave numbers to parts that had none: 2
Connections:
- net labels added: GND_3V3, GND_3v3, SD3, SD4
- net labels removed: CLK, DAT0
- wire segments 137 -> 145
- no-connect marks 2 -> 21

Commit message: :zap: Improving PCB performance
Changed lines of the file:
@@
 Wire Wire Line
 	1800 2800 1500 2800
+Text Label 1500 2800 0    50   ~ 0
+SD3
 Text Label 1500 2700 0    50   ~ 0
-SD3
-Text Label 1500 2800 0    50   ~ 0
 SD4
 NoConn ~ 3400 3500
